Commit message: 更新机器人模型，忽略 ROS 2 编译产物和日志

File: src/warehouse_description/urdf/warehouse_robot.urdf.xacro (robot description, xacro)
@@ -20,5 +20,5 @@
   <link name="base_link">
     <visual>
-      <origin xyz="0 0 ${body_h / 2.0}"/>
+      <origin xyz="0 0 ${0.17 + body_h / 2.0}"/>
       <geometry>
         <box size="${body_l} ${body_w} ${body_h}"/>
@@ -27,5 +27,5 @@
     </visual>
     <collision>
-      <origin xyz="0 0 ${body_h / 2.0}"/>
+      <origin xyz="0 0 ${0.17 + body_h / 2.0}"/>
       <geometry>
         <box size="${body_l} ${body_w} ${body_h}"/>
@@ -33,9 +33,9 @@
     </collision>
     <inertial>
-      <origin xyz="0 0 ${body_h / 2.0}"/>
+      <origin xyz="0 0 ${0.17 + body_h / 2.0}"/>
       <mass value="20.0"/>
-      <inertia ixx="1.0" ixy="0" ixz="0"
-               iyy="1.0" iyz="0"
-               izz="1.0"/>
+      <inertia ixx="0.441667" ixy="0" ixz="0"
+               iyy="0.704167" iyz="0"
+               izz="0.937500"/>
     </inertial>
   </link>
@@ -54,4 +54,11 @@
       </geometry>
     </collision>
+  <inertial>
+  <origin xyz="0 0 0"/>
+  <mass value="1.0"/>
+  <inertia ixx="0.00173333" ixy="0" ixz="0"
+           iyy="0.00173333" iyz="0"
+           izz="0.0032"/>
+  </inertial>
   </link>
   <gazebo reference="left_wheel_link">
@@ -62,5 +69,5 @@
     <parent link="base_link"/>
     <child link="left_wheel_link"/>
-    <origin xyz="0 0.25 0.08"
+    <origin xyz="0.10 0.25 0.18"
             rpy="1.5708 0 0"/>
     <axis xyz="0 0 1"/>
@@ -79,4 +86,11 @@
       </geometry>
     </collision>
+  <inertial>
+  <origin xyz="0 0 0"/>
+  <mass value="1.0"/>
+  <inertia ixx="0.00173333" ixy="0" ixz="0"
+           iyy="0.00173333" iyz="0"
+           izz="0.0032"/>
+  </inertial>
   </link>
   <gazebo reference="right_wheel_link">
@@ -87,5 +101,5 @@
     <parent link="base_link"/>
     <child link="right_wheel_link"/>
-    <origin xyz="0 -0.25 0.08"
+    <origin xyz="0.10 -0.25 0.18"
             rpy="1.5708 0 0"/>
     <axis xyz="0 0 1"/>
@@ -104,4 +118,11 @@
       </geometry>
     </collision>
+  <inertial>
+  <origin xyz="0 0 0"/>
+  <mass value="0.2"/>
+  <inertia ixx="0.000128" ixy="0" ixz="0"
+           iyy="0.000128" iyz="0"
+           izz="0.000128"/>
+  </inertial>
   </link>
   <gazebo reference="caster_wheel_link">
@@ -112,5 +133,5 @@
     <parent link="base_link"/>
     <child link="caster_wheel_link"/>
-    <origin xyz="-0.22 0 0.04"/>
+    <origin xyz="-0.22 0 0.14"/>
   </joint>
   <!-- 激光雷达 -->
@@ -127,5 +148,5 @@
     <parent link="base_link"/>
     <child link="laser_link"/>
-    <origin xyz="0.20 0 0.30"/>
+    <origin xyz="0.20 0 0.46"/>
   </joint>
   <!-- IMU -->
@@ -142,5 +163,5 @@
     <parent link="base_link"/>
     <child link="imu_link"/>
-    <origin xyz="0 0 0.20"/>
+    <origin xyz="0 0 0.30"/>
   </joint>
 </robot>

Commit message: 阶段1：加差速驱动插件、仓库 world 与 Gazebo 启动 launch

File: src/warehouse_description/urdf/warehouse_robot.urdf.xacro (robot description, xacro)
@@ -7,5 +7,5 @@
   <xacro:property name="wheel_r" value="0.08"/>
   <xacro:property name="wheel_w" value="0.04"/>
-  <xacro:property name="wheel_track" value="0.42"/>
+  <xacro:property name="wheel_track" value="0.50"/>
   <material name="blue">
     <color rgba="0.1 0.3 0.8 1.0"/>
@@ -64,4 +64,6 @@
   <gazebo reference="left_wheel_link">
   <material>Gazebo/Black</material>
+  <mu1>1.5</mu1>
+  <mu2>1.5</mu2>
   </gazebo>
   <joint name="left_wheel_joint"
@@ -69,6 +71,6 @@
     <parent link="base_link"/>
     <child link="left_wheel_link"/>
-    <origin xyz="0.10 0.25 0.18"
-            rpy="1.5708 0 0"/>
+    <origin xyz="0.10 ${wheel_track / 2.0} 0.18"
+            rpy="-1.5708 0 0"/>
     <axis xyz="0 0 1"/>
   </joint>
@@ -96,4 +98,6 @@
   <gazebo reference="right_wheel_link">
   <material>Gazebo/Black</material>
+  <mu1>1.5</mu1>
+  <mu2>1.5</mu2>
   </gazebo>
   <joint name="right_wheel_joint"
@@ -101,6 +105,6 @@
     <parent link="base_link"/>
     <child link="right_wheel_link"/>
-    <origin xyz="0.10 -0.25 0.18"
-            rpy="1.5708 0 0"/>
+    <origin xyz="0.10 -${wheel_track / 2.0} 0.18"
+            rpy="-1.5708 0 0"/>
     <axis xyz="0 0 1"/>
   </joint>
@@ -128,4 +132,6 @@
   <gazebo reference="caster_wheel_link">
   <material>Gazebo/Black</material>
+  <mu1>0.001</mu1>
+  <mu2>0.001</mu2>
   </gazebo>
   <joint name="caster_wheel_joint"
@@ -165,3 +171,33 @@
     <origin xyz="0 0 0.30"/>
   </joint>
+  <!-- Gazebo 不读 URDF 的 material，需要单独指定预置材质 -->
+  <gazebo reference="base_link">
+    <material>Gazebo/Blue</material>
+  </gazebo>
+  <gazebo reference="laser_link">
+    <material>Gazebo/Red</material>
+  </gazebo>
+  <gazebo reference="imu_link">
+    <material>Gazebo/Black</material>
+  </gazebo>
+  <!-- 差速驱动：订阅 cmd_vel，发布 odom 并广播 odom -> base_link -->
+  <gazebo>
+    <plugin name="warehouse_diff_drive" filename="libgazebo_ros_diff_drive.so">
+      <update_rate>30.0</update_rate>
+      <left_joint>left_wheel_joint</left_joint>
+      <right_joint>right_wheel_joint</right_joint>
+      <wheel_separation>${wheel_track}</wheel_separation>
+      <wheel_diameter>${2 * wheel_r}</wheel_diameter>
+      <max_wheel_torque>30.0</max_wheel_torque>
+      <max_wheel_acceleration>2.0</max_wheel_acceleration>
+      <command_topic>cmd_vel</command_topic>
+      <publish_odom>true</publish_odom>
+      <publish_odom_tf>true</publish_odom_tf>
+      <publish_wheel_tf>false</publish_wheel_tf>
+      <odometry_topic>odom</odometry_topic>
+      <odometry_source>world</odometry_source>
+      <odometry_frame>odom</odometry_frame>
+      <robot_base_frame>base_link</robot_base_frame>
+    </plugin>
+  </gazebo>
 </robot>

Commit message: imu_link 补 inertial，修复 /imu 零帧

File: src/warehouse_description/urdf/warehouse_robot.urdf.xacro (robot description, xacro)
@@ -164,4 +164,13 @@
       <material name="red"/>
     </visual>
+    <!-- 不写 inertial 时 Gazebo 按视觉体积+密度 1 推出 4.8e-5 kg，与 20 kg 车身差 40 万倍，
+         这个 link 在物理引擎里等于不存在，IMU 传感器于是永远不发数据（发布者有、零帧） -->
+    <inertial>
+      <origin xyz="0 0 0"/>
+      <mass value="0.05"/>
+      <inertia ixx="0.0000083" ixy="0" ixz="0"
+               iyy="0.0000167" iyz="0"
+               izz="0.0000217"/>
+    </inertial>
   </link>
   <joint name="imu_joint"
